File: pcbs/power_distribution/_autosave-power_distribution.kicad_pcb (KiCad board)
At the start: 2 copper layers, 29 parts, among them J1 Conn_01x02, J10 Conn_01x06, J11 Conn_01x06, J12 Conn_01x06, J13 Conn_01x06, J14 Conn_01x06, J15 Conn_01x06, J16 Conn_01x06, J2 Conn_01x02, J3 Conn_01x02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

Commit message: add CAN test scripts
Parts:
- added REF**: MODULE_RASPBERRY_PI_4B_4GB, General:MODULE_RASPBERRY_PI_4B_4GB, F.Cu at (173.0, 134.5)
- JP1, JP2, JP3, JP4: moved to B.Cu
- moved MOD1 140.8 mm to (273.3, 209.8)
- moved PS1 132.5 mm to (318.5, 196.2)
- moved H1 101.5 mm to (275.0, 75.8)
- moved H2 101.5 mm to (275.0, 82.4)
- moved H3 101.5 mm to (275.0, 89.0)
- moved H4 101.5 mm to (275.0, 95.5)
- moved JP1 73.2 mm to (121.7, 179.9), turned to 180 degrees
- moved JP3 73.2 mm to (121.7, 176.3), turned to 180 degrees
- moved JP4 73.2 mm to (121.7, 187.0), turned to 180 degrees
- moved JP2 73.2 mm to (121.7, 183.4), turned to 180 degrees
- moved J4 55.3 mm to (154.0, 92.5)
- moved J1 34.9 mm to (173.0, 92.0)
- moved J16 19.5 mm to (205.5, 309.5)
- moved J11 19.3 mm to (133.0, 309.5)
- moved J12 18.8 mm to (147.5, 309.5)
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Other:
- board outline added: 120 x 250 mm
