File: pcbs/power_distribution/power_distribution.kicad_sch (KiCad schematic)
At the start: 18 parts, among them J1 Conn_01x06, J2 Conn_01x06, J3 Conn_01x06, J4 Conn_01x06, J5 Conn_01x06, J6 Conn_01x06, J7 Conn_01x02, J8 Conn_01x02, J9 Conn_01x02

Commit message: add CAN test scripts
Parts:
- removed J8: Conn_01x02, Connector_AMASS:AMASS_XT30U-M_1x02_P5.0mm_Vertical, symbol Connector_Generic:Conn_01x02
- added J11, J12, J13, J14, J15, J16: Conn_01x06, Connector_JST:JST_ZH_B6B-ZR_1x06_P1.50mm_Vertical, symbol Connector_Generic:Conn_01x06
- added J3, J4: Conn_01x02, Connector_JST:JST_ZH_B2B-ZR_1x02_P1.50mm_Vertical, symbol Connector_Generic:Conn_01x02
- added JP2, JP4: SolderJumper_2_Open, Jumper:SolderJumper-2_P1.3mm_Open_Pad1.0x1.5mm, symbol Jumper:SolderJumper_2_Open
- added MOD1: BNO055_Module, General:BNO055 Module, symbol General:BNO055_Module
- added PS1: SHHD003A0A41Z, General:SHHD003A0A41Z, symbol General:SHHD003A0A41Z
- renumbered J9 to J1, J6 to J10, J7 to J2, J1 to J5, J2 to J6, J3 to J7, J4 to J8, J5 to J9, JP2 to JP1, JP1 to JP3
Connections:
- net +BATT: now also J11.5 (Pin_5), J11.6 (Pin_6), J12.5 (Pin_5), J12.6 (Pin_6), J13.5 (Pin_5), J13.6 (Pin_6), J14.5 (Pin_5), J14.6 (Pin_6), J15.5 (Pin_5), J15.6 (Pin_6), J16.5 (Pin_5), J16.6 (Pin_6)
- net CAN1 HIGH: now also J11.2 (Pin_2), J12.2 (Pin_2), J13.2 (Pin_2), J3.1 (Pin_1), JP2.1 (A)
- net CAN2 HIGH: now also J14.2 (Pin_2), J15.2 (Pin_2), J16.2 (Pin_2), J4.1 (Pin_1), JP2.2 (B)
- net CAN2 LOW: now also J11.1 (Pin_1), J12.1 (Pin_1), J13.1 (Pin_1), J14.1 (Pin_1), J15.1 (Pin_1), J16.1 (Pin_1), J3.2 (Pin_2), J4.2 (Pin_2), JP4.1 (A), JP4.2 (B)
- net GND: now also J11.3 (Pin_3), J11.4 (Pin_4), J12.3 (Pin_3), J12.4 (Pin_4), J13.3 (Pin_3), J13.4 (Pin_4), J14.3 (Pin_3), J14.4 (Pin_4), J15.3 (Pin_3), J15.4 (Pin_4), J16.3 (Pin_3), J16.4 (Pin_4)
Other:
- moved on the sheet: BH1, BH2, BH3, H1, H2, H3, H4, J1, J10, J2, J5, J6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

Commit message: PCB update
Parts:
- removed BH1, BH2, BH3: 2x_18650_Li-ion_Holder, General:2x_18650_battery_holder, symbol General:2x_18650_battery_holder
- removed J1, J2, J4: Conn_01x02, Connector_JST:JST_ZH_B2B-ZR_1x02_P1.50mm_Vertical, symbol Connector_Generic:Conn_01x02
- removed MOD1: BNO055_Module, General:BNO055 Module, symbol General:BNO055_Module
- added BH1, BH2: 2x_18650_Li-ion_Holder, General:3x_18650_battery_holder, symbol General:3x_18650_battery_holder
- added D1: LED, LED_SMD:LED_1206_3216Metric, symbol Device:LED
- added H5, H6, H7, H8: MountingHole, MountingHole:MountingHole_2.5mm_Pad_TopBottom, symbol Mechanical:MountingHole
- added J1, J2, J20, J21: Conn_01x03, symbol Connector_Generic:Conn_01x03
- added J18, J19: XT60PW-M, Connectors:AMASS_XT60PW-M, symbol Connectors:XT60PW-M
- added R1: R_Small_US, Resistor_SMD:R_1206_3216Metric, symbol Device:R_Small_US
- added SBC1: ~, General:RASPBERRY_PI_4B - Footprint Only, symbol General:Raspberry Pi - Footprint_Only
- added SW1: SW_SPST, symbol Switch:SW_SPST
- J3: footprint Connector_JST:JST_ZH_B2B-ZR_1x02_P1.50mm_Vertical -> (none)
Connections:
- net +BATT: now also J19.1 (+), SW1.1 (A); no longer J10.5 (Pin_5), J10.6 (Pin_6), J5.5 (Pin_5), J5.6 (Pin_6), J6.5 (Pin_5), J6.6 (Pin_6), J7.5 (Pin_5), J7.6 (Pin_6), J8.5 (Pin_5), J8.6 (Pin_6), J9.5 (Pin_5), J9.6 (Pin_6)
- net CAN1 HIGH: now also J1.1 (Pin_1), J20.1 (Pin_1); no longer J3.1 (Pin_1)
- net CAN2 HIGH: now also J2.1 (Pin_1), J21.1 (Pin_1)
- net CAN2 LOW: now also J1.2 (Pin_2), J2.2 (Pin_2), J20.2 (Pin_2), J21.2 (Pin_2); no longer J3.2 (Pin_2)
- net GND: now also PS1.2 (VIN-), J1.3 (Pin_3), J18.2 (-), J19.2 (-), J2.3 (Pin_3), J20.3 (Pin_3), J21.3 (Pin_3), R1.2
- net +MOT: now reaches PS1.1 (VIN+)
- net +MOT: now also J10.5 (Pin_5), J10.6 (Pin_6), J5.5 (Pin_5), J5.6 (Pin_6), J6.5 (Pin_5), J6.6 (Pin_6), J7.5 (Pin_5), J7.6 (Pin_6), J8.5 (Pin_5), J8.6 (Pin_6), J9.5 (Pin_5), J9.6 (Pin_6), D1.2 (A), J18.1 (+), SW1.2 (B)
- net at PS1.4 (VOUT-): now also J3.2 (Pin_2)
- net at PS1.6 (VOUT+): now also J3.1 (Pin_1)
- new net: D1.1 (K), R1.1
Other:
- note added: "Isolated Power Used for CTRL Electronics Only"
- moved on the sheet: H1, H2, H3, H4, PS1

Commit message: PCB update.
Parts:
- removed BH1, BH2: 2x_18650_Li-ion_Holder, General:3x_18650_battery_holder, symbol General:3x_18650_battery_holder
- removed H1, H2, H3, H4, H5, H6, H7, H8: MountingHole, MountingHole:MountingHole_2.5mm_Pad_TopBottom, symbol Mechanical:MountingHole
- removed J18, J19: XT60PW-M, Connectors:AMASS_XT60PW-M, symbol Connectors:XT60PW-M
- removed PS1: SHHD003A0A41Z, General:SHHD003A0A41Z, symbol General:SHHD003A0A41Z
- added BATT1: ~, General:18650 6S Battery Pack - Footprint Only, symbol General:18650 6s Battery Pack - Footprint Only
- added J4: AMASS Connector, power-and-batteries:AMASS_XT30U-M_1x02_P5.0mm_Vertical, symbol power-and-batteries:AMASS Connector
- added U1: SCW12B-05, SCW12B-05_MWU, symbol power-and-batteries:SCW12B-05
- J1, J2, J20, J21: footprint (none) -> Connector_JST:JST_ZH_B3B-ZR_1x03_P1.50mm_Vertical
- J3: footprint (none) -> TerminalBlock_Phoenix:TerminalBlock_Phoenix_MKDS-1,5-2_1x02_P5.00mm_Horizontal
- SW1: footprint (none) -> switches-and-buttons:CRE22F4DBBNE
Connections:
- net +MOT is gone; now on net +BATT: D1.2 (A), J10.5 (Pin_5), J10.6 (Pin_6), J5.5 (Pin_5), J5.6 (Pin_6), J6.5 (Pin_5), J6.6 (Pin_6), J7.5 (Pin_5), J7.6 (Pin_6), J8.5 (Pin_5), J8.6 (Pin_6), J9.5 (Pin_5), J9.6 (Pin_6), SW1.2 (B)
- net +BATT: now also U1.22 (+VIN), U1.23 (+VIN); no longer SW1.1 (A)
- net CAN1 HIGH: no longer J20.1 (Pin_1), J5.2 (Pin_2), J6.2 (Pin_2), J7.2 (Pin_2), JP1.1 (A)
- net CAN2 HIGH: no longer J10.2 (Pin_2), J21.1 (Pin_1), J8.2 (Pin_2), J9.2 (Pin_2), JP1.2 (B)
- net CAN2 LOW: no longer J1.2 (Pin_2), J10.1 (Pin_1), J11.1 (Pin_1), J12.1 (Pin_1), J13.1 (Pin_1), J20.2 (Pin_2), J21.2 (Pin_2), J5.1 (Pin_1), J6.1 (Pin_1), J7.1 (Pin_1), J8.1 (Pin_1), J9.1 (Pin_1), JP3.1 (A), JP3.2 (B), JP4.1 (A)
- net GND: now also J4.1 (-), U1.2 (-VIN), U1.3 (-VIN)
- net ISO 5vDC GND: now reaches J3.1 (Pin_1)
- net ISO 5vDC GND: now also U1.14 (+VOUT)
- net ISO 5vDC+: now reaches J3.2 (Pin_2)
- net ISO 5vDC+: now also U1.16 (-VOUT)
- new net: J4.2 (+), SW1.1 (A)
- new net CAN1 LOW: J1.2 (Pin_2), J11.1 (Pin_1), J12.1 (Pin_1), J13.1 (Pin_1), JP4.1 (A)
- new net CAN3 HIGH: J20.1 (Pin_1), J5.2 (Pin_2), J6.2 (Pin_2), J7.2 (Pin_2), JP1.1 (A)
- new net CAN3 LOW: J20.2 (Pin_2), J5.1 (Pin_1), J6.1 (Pin_1), J7.1 (Pin_1), JP3.1 (A)
- new net CAN4 HIGH: J10.2 (Pin_2), J21.1 (Pin_1), J8.2 (Pin_2), J9.2 (Pin_2), JP1.2 (B)
- new net CAN4 LOW: J10.1 (Pin_1), J21.2 (Pin_2), J8.1 (Pin_1), J9.1 (Pin_1), JP3.2 (B)
- no-connect marks 0 -> 1
Other:
- note added: "BACK LEFT"
- note added: "BACK RIGHT"
- note added: "Battery In"
- note added: "FRONT LEFT"
- note added: "FRONT RIGHT"
- moved on the sheet: D1, J1, J10, J11, J12, J13, J14, J15, J16, J2, J20, J21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

Commit message: PCB update.
Other:
- moved on the sheet: BATT1, D1, R1, SBC1
Changed lines of the file:
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@@
 	(wire
 		(pts
-			(xy 43.18 247.65) (xy 43.18 251.46)
+			(xy 58.42 231.14) (xy 58.42 234.95)
 		)
 		(stroke
@@
 	(wire
 		(pts
-			(xy 43.18 240.03) (xy 43.18 242.57)
+			(xy 58.42 223.52) (xy 58.42 226.06)
 		)
 		(stroke
@@
 	(wire
 		(pts
-			(xy 43.18 229.87) (xy 43.18 232.41)
+			(xy 58.42 213.36) (xy 58.42 215.9)
 		)
 		(stroke
@@
 	(symbol
 		(lib_id "General:18650 6s Battery Pack - Footprint Only")
-		(at 109.22 238.76 0)
+		(at 124.46 222.25 0)
 		(unit 1)
 		(exclude_from_sim no)
@@
 		(dnp no)
 		(property "Reference" "BATT1"
-			(at 106.934 250.698 0)
+			(at 122.174 234.188 0)
 			(effects
 				(font
@@
 		)
 		(property "Value" "~"
-			(at 109.22 238.76 0)
+			(at 124.46 222.25 0)
 			(effects
 				(font
@@
 		)
 		(property "Footprint" "General:18650 6S Battery Pack - Footprint Only"
-			(at 109.22 238.76 0)
+			(at 124.46 222.25 0)
 			(effects
 				(font
@@
 		)
 		(property "Datasheet" ""
-			(at 109.22 238.76 0)
+			(at 124.46 222.25 0)
 			(effects
 				(font
@@
 		)
 		(property "Description" "DIY with BMS"
-			(at 109.22 238.76 0)
+			(at 124.46 222.25 0)
 			(effects
 				(font
@@
 	(symbol
 		(lib_id "Device:R_Small_US")
-		(at 43.18 245.11 0)
+		(at 58.42 228.6 0)
 		(unit 1)
 		(exclude_from_sim no)
@@
 		(fields_autoplaced yes)
 		(property "Reference" "R1"
-			(at 45.72 245.1099 0)
+			(at 60.96 228.5999 0)
 			(effects
 				(font
@@
 		)
 		(property "Value" "R_Small_US"
-			(at 45.72 246.3799 0)
+			(at 60.96 229.8699 0)
 			(effects
 				(font
@@
 		)
 		(property "Footprint" "Resistor_SMD:R_1206_3216Metric"
-			(at 43.18 245.11 0)
+			(at 58.42 228.6 0)
 			(effects
 				(font
@@
 		)
 		(property "Datasheet" "~"
-			(at 43.18 245.11 0)
+			(at 58.42 228.6 0)
 			(effects
 				(font
@@
 		)
 		(property "Description" "Resistor, small US symbol"
-			(at 43.18 245.11 0)
+			(at 58.42 228.6 0)
 			(effects
 				(font
@@
 	(symbol
 		(lib_id "power:GND")
-		(at 43.18 251.46 0)
+		(at 58.42 234.95 0)
 		(unit 1)
 		(exclude_from_sim no)
@@
 		(fields_autoplaced yes)
 		(property "Reference" "#PWR014"
-			(at 43.18 257.81 0)
+			(at 58.42 241.3 0)
 			(effects
 				(font
@@
 		)
 		(property "Value" "GND"
-			(at 43.18 256.54 0)
+			(at 58.42 240.03 0)
 			(effects
 				(font
@@
 		)
 		(property "Footprint" ""
-			(at 43.18 251.46 0)
+			(at 58.42 234.95 0)
 			(effects
 				(font
@@
 		)
 		(property "Datasheet" ""
-			(at 43.18 251.46 0)
+			(at 58.42 234.95 0)
 			(effects
 				(font
@@
 		)
 		(property "Description" "Power symbol creates a global label with name \"GND\" , ground"
-			(at 43.18 251.46 0)
+			(at 58.42 234.95 0)
 			(effects
 				(font
@@
 	(symbol
 		(lib_id "General:Raspberry Pi - Footprint_Only")
-		(at 74.93 238.76 0)
+		(at 90.17 222.25 0)
 		(unit 1)
 		(exclude_from_sim no)
@@
 		(fields_autoplaced yes)
 		(property "Reference" "SBC1"
-			(at 85.09 244.4749 0)
+			(at 100.33 227.9649 0)
 			(effects
 				(font
@@
 		)
 		(property "Value" "~"
-			(at 85.09 246.38 0)
+			(at 100.33 229.87 0)
 			(effects
 				(font
@@
 		)
 		(property "Footprint" "General:RASPBERRY_PI_4B - Footprint Only"
-			(at 74.93 238.76 0)
+			(at 90.17 222.25 0)
 			(effects
 				(font
@@
 		)
 		(property "Datasheet" ""
-			(at 74.93 238.76 0)
+			(at 90.17 222.25 0)
 			(effects
 				(font
@@
 		)
 		(property "Description" ""
-			(at 74.93 238.76 0)
+			(at 90.17 222.25 0)
 			(effects
 				(font
@@
 	(symbol
 		(lib_id "power:+BATT")
-		(at 43.18 229.87 0)
+		(at 58.42 213.36 0)
 		(unit 1)
 		(exclude_from_sim no)
@@
 		(fields_autoplaced yes)
 		(property "Reference" "#PWR05"
-			(at 43.18 233.68 0)
+			(at 58.42 217.17 0)
 			(effects
 				(font
@@
 		)
 		(property "Value" "+BATT"
-			(at 43.18 224.79 0)
+			(at 58.42 208.28 0)
 			(effects
 				(font
@@
 		)
 		(property "Footprint" ""
-			(at 43.18 229.87 0)
+			(at 58.42 213.36 0)
 			(effects
 				(font
@@
 		)
 		(property "Datasheet" ""
-			(at 43.18 229.87 0)
+			(at 58.42 213.36 0)
 			(effects
 				(font
@@
 		)
 		(property "Description" "Power symbol creates a global label with name \"+BATT\""
-			(at 43.18 229.87 0)
+			(at 58.42 213.36 0)
 			(effects
 				(font
@@
 	(symbol
 		(lib_id "Device:LED")
-		(at 43.18 236.22 90)
+		(at 58.42 219.71 90)
 		(unit 1)
 		(exclude_from_sim no)
@@
 		(fields_autoplaced yes)
 		(property "Reference" "D1"
-			(at 46.99 236.5374 90)
+			(at 62.23 220.0274 90)
 			(effects
 				(font
@@
 		)
 		(property "Value" "LED"
-			(at 46.99 239.0774 90)
+			(at 62.23 222.5674 90)
 			(effects
 				(font
@@
 		)
 		(property "Footprint" "LED_SMD:LED_1206_3216Metric"
-			(at 43.18 236.22 0)
+			(at 58.42 219.71 0)
 			(effects
 				(font
@@
 		)
 		(property "Datasheet" "~"
-			(at 43.18 236.22 0)
+			(at 58.42 219.71 0)
 			(effects
 				(font
@@
 		)
 		(property "Description" "Light emitting diode"
-			(at 43.18 236.22 0)
+			(at 58.42 219.71 0)
 			(effects
 				(font
