File: pcbs/power_distribution/power_distribution.kicad_pcb (KiCad board)
At the start: 2 copper layers, 29 parts, among them J1 Conn_01x02, J10 Conn_01x06, J11 Conn_01x06, J12 Conn_01x06, J13 Conn_01x06, J14 Conn_01x06, J15 Conn_01x06, J16 Conn_01x06, J2 Conn_01x02, J3 Conn_01x02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

Commit message: PCB update
Parts:
- removed BH3: 2x_18650_Li-ion_Holder, General:2x_18650_battery_holder
- removed MOD1: BNO055_Module, General:BNO055 Module
- added SBC1: ~, General:RASPBERRY_PI_4B - Footprint Only, F.Cu at (170.5, 145.5)
- BH1, BH2: footprint General:2x_18650_battery_holder -> General:3x_18650_battery_holder
- JP1, JP2, JP3, JP4, PS1: moved to B.Cu
- moved H1 158.8 mm to (103.5, 237.5)
- moved H2 143.9 mm to (102.5, 226.5)
- moved JP1 114.7 mm to (223.3, 191.9), turned to 180 degrees
- moved JP3 114.7 mm to (223.3, 188.3), turned to 180 degrees
- moved JP4 114.7 mm to (223.3, 199.0), turned to 180 degrees
- moved JP2 114.7 mm to (223.3, 195.4), turned to 180 degrees
- moved H4 101.5 mm to (275.0, 95.5)
- moved J4 57.2 mm to (222.5, 173.0)
- moved J1 55.9 mm to (222.5, 163.5)
- moved BH2 55.8 mm to (134.0, 252.5)
- moved H3 48.5 mm to (224.0, 110.0)
- moved BH1 40.3 mm to (134.0, 185.2)
- moved J3 35.9 mm to (222.8, 132.6)
- moved J2 35.3 mm to (222.8, 123.0)
- moved PS1 29.3 mm to (169.5, 144.0), turned to 90 degrees
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Other:
- board outline added: 120 x 250 mm

Commit message: PCB update.
Parts:
- removed BH1, BH2: 2x_18650_Li-ion_Holder, General:3x_18650_battery_holder
- removed H1, H2, H3, H4: MountingHole, MountingHole:MountingHole_2.5mm_Pad_TopBottom
- removed PS1: SHHD003A0A41Z, General:SHHD003A0A41Z
- added BATT1: ~, General:18650 6S Battery Pack - Footprint Only, F.Cu at (140.5, 225.0)
- added D1: LED, LED_SMD:LED_1206_3216Metric, F.Cu at (140.8, 207.1)
- added J20: Conn_01x03, Connector_JST:JST_ZH_B3B-ZR_1x03_P1.50mm_Vertical, F.Cu at (202.0, 147.0)
- added J21: Conn_01x03, Connector_JST:JST_ZH_B3B-ZR_1x03_P1.50mm_Vertical, F.Cu at (202.0, 156.0)
- added R1: R_Small_US, Resistor_SMD:R_1206_3216Metric, F.Cu at (145.3, 207.0)
- added SW1: SW_SPST, switches-and-buttons:CRE22F4DBBNE, F.Cu at (170.0, 215.5)
- added U1: SCW12B-05, power-and-batteries:SCW12B-05_MWU, B.Cu at (177.2, 146.1)
- J1, J2: value Conn_01x02 -> Conn_01x03; footprint Connector_JST:JST_ZH_B2B-ZR_1x02_P1.50mm_Vertical -> Connector_JST:JST_ZH_B3B-ZR_1x03_P1.50mm_Vertical
- J3: footprint Connector_JST:JST_ZH_B2B-ZR_1x02_P1.50mm_Vertical -> TerminalBlock_Phoenix:TerminalBlock_Phoenix_MKDS-1,5-2_1x02_P5.00mm_Horizontal
- J4: value Conn_01x02 -> AMASS Connector; footprint Connector_JST:JST_ZH_B2B-ZR_1x02_P1.50mm_Vertical -> power-and-batteries:AMASS_XT30U-M_1x02_P5.0mm_Vertical
- moved J11 236.1 mm to (138.5, 79.0), turned to -90 degrees
- moved J16 236.0 mm to (202.5, 79.0), turned to -90 degrees
- moved J12 236.0 mm to (151.3, 79.0), turned to -90 degrees
- moved J15 236.0 mm to (189.7, 79.0), turned to -90 degrees
- moved J13 236.0 mm to (164.1, 79.0), turned to -90 degrees
- moved J14 236.0 mm to (176.9, 79.0), turned to -90 degrees
- moved J10 227.6 mm to (201.5, 311.0)
- moved J9 227.5 mm to (188.7, 311.0)
- moved J5 227.5 mm to (137.5, 311.0)
- moved J8 227.5 mm to (175.9, 311.0)
- moved J6 227.5 mm to (150.3, 311.0)
- moved J7 227.5 mm to (163.1, 311.0)
- moved JP3 135.0 mm to (171.5, 313.0), turned to 0 degrees
- moved JP4 133.1 mm to (168.0, 78.0), turned to 0 degrees
- moved JP1 130.9 mm to (168.0, 310.5), turned to 0 degrees
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Connections:
- J1 pad 2: /CAN2 LOW -> /CAN1 LOW
- J10 pad 1: /CAN2 LOW -> /CAN4 LOW
- J10 pad 2: /CAN2 HIGH -> /CAN4 HIGH
- J11 pad 1: /CAN2 LOW -> /CAN1 LOW
- J12 pad 1: /CAN2 LOW -> /CAN1 LOW
- J13 pad 1: /CAN2 LOW -> /CAN1 LOW
- J3 pad 1: /CAN1 HIGH -> /ISO 5vDC GND
- J3 pad 2: /CAN2 LOW -> /ISO 5vDC+
- J4 pad 1: /CAN2 HIGH -> GND
- J4 pad 2: /CAN2 LOW -> Net-(J4-+)
- J5 pad 1: /CAN2 LOW -> /CAN3 LOW
- J5 pad 2: /CAN1 HIGH -> /CAN3 HIGH
- J6 pad 1: /CAN2 LOW -> /CAN3 LOW
- J6 pad 2: /CAN1 HIGH -> /CAN3 HIGH
- J7 pad 1: /CAN2 LOW -> /CAN3 LOW
- J7 pad 2: /CAN1 HIGH -> /CAN3 HIGH
- J8 pad 1: /CAN2 LOW -> /CAN4 LOW
- J8 pad 2: /CAN2 HIGH -> /CAN4 HIGH
- J9 pad 1: /CAN2 LOW -> /CAN4 LOW
- J9 pad 2: /CAN2 HIGH -> /CAN4 HIGH
- JP1 pad 1: /CAN1 HIGH -> /CAN3 HIGH
- JP1 pad 2: /CAN2 HIGH -> /CAN4 HIGH
- JP3 pad 1: /CAN2 LOW -> /CAN3 LOW
- JP3 pad 2: /CAN2 LOW -> /CAN4 LOW
- JP4 pad 1: /CAN2 LOW -> /CAN1 LOW
Other:
- board size 120 x 250 mm -> 120 x 240 mm
- board text added: "+"
- board text added: "-"
- board text added: "BACK LEFT"
- board text added: "BACK RIGHT"
- board text added: "BATTERY"
- board text added: "CAN1"
- board text added: "CAN2"
- board text added: "CAN3"
- board text added: "CAN4"
- board text added: "FRONT LEFT"
- board text added: "FRONT RIGHT"
- board text added: "ISO 5vDC"
- board text added: "RASPBERRY PI"
- board text added: "SCW12B-05 DC-DC ISOLATED"

Commit message: PCB update.
Other:
- outline, holes or cut-outs redrawn

Commit message: PCB update.
Parts:
- U1: moved to F.Cu
- moved U1 61.2 mm to (156.1, 203.5), turned to 90 degrees
- moved D1 57.4 mm to (198.0, 202.2), turned to -90 degrees
- moved J3 48.5 mm to (192.8, 191.0), turned to 90 degrees
- moved R1 48.4 mm to (193.5, 202.2), turned to -90 degrees
- moved J2 14.0 mm to (201.6, 106.0)
- moved J21 7.52 mm to (201.5, 148.5)
- moved J20 7.51 mm to (201.6, 139.5)
- moved SBC1 7.00 mm to (169.0, 139.0)
- moved J4 6.08 mm to (193.0, 212.0)
- moved J1 5.02 mm to (201.6, 97.0)
- moved BATT1 2.50 mm to (140.5, 227.5)
- moved SW1 0.05 mm to (170.1, 215.5), turned to 0 degrees
Routing:
- net +BATT: track 0.00 -> 626.8 mm
- net /CAN3 LOW: track 0.00 -> 263.3 mm, vias 0 -> 2
- net /CAN3 HIGH: track 0.00 -> 254.8 mm, vias 0 -> 2
- net /CAN4 LOW: track 0.00 -> 206.6 mm
- net /CAN4 HIGH: track 0.00 -> 205.2 mm
- net Net-(J4-+): track 0.00 -> 110.6 mm
- net /CAN1 LOW: track 0.00 -> 75.0 mm, vias 0 -> 2
- net /CAN1 HIGH: track 0.00 -> 73.9 mm, vias 0 -> 1
- net /CAN2 LOW: track 0.00 -> 63.9 mm
- net /CAN2 HIGH: track 0.00 -> 60.3 mm
- net /ISO 5vDC+: track 0.00 -> 22.3 mm
- net /ISO 5vDC GND: track 0.00 -> 12.5 mm
- net Net-(D1-K): track 0.00 -> 4.53 mm
- net GND: track 0.00 -> 3.54 mm, vias 0 -> 1
- added copper zone on F.Cu, net +BATT
- added copper zone on B.Cu, net GND
Other:
- board size 120 x 240 mm -> 74 x 240 mm
- board text added: "ElectroPup Power Carrier metaphasiclabs.com 09/2024"
