File: pcbs/power_distribution/aux-board/_autosave-aux-board.kicad_pcb (KiCad board)
At the start: 2 copper layers, 85 x 56 mm, 8 parts, among them J5 Raspberry Pi - Hat Template -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, SW1 SW_Push, SW2 SW_Push, U1 YAAJ_WeAct_BlackPill_Part_Like

Commit message: PCB update.
Parts:
- added J1: Conn_01x03, Connector_JST:JST_ZH_B3B-ZR_1x03_P1.50mm_Vertical, F.Cu at (140.5, 74.9)
- added J2: Conn_01x03, Connector_JST:JST_ZH_B3B-ZR_1x03_P1.50mm_Vertical, F.Cu at (140.5, 80.5)
- added J3: Conn_01x03, Connector_JST:JST_ZH_B3B-ZR_1x03_P1.50mm_Vertical, F.Cu at (140.5, 86.0)
- added J6: Conn_01x02, TerminalBlock_Phoenix:TerminalBlock_Phoenix_PT-1,5-2-5.0-H_1x02_P5.00mm_Horizontal, F.Cu at (24.0, 80.0)
- moved MOD1 19.0 mm to (95.6, 57.1), turned to -90 degrees
Connections:
- J5 pad 02: unconnected-(J5-5V_PWR-Pad02) -> +5V
- J5 pad 04: unconnected-(J5-5V_PWR-Pad04) -> +5V
- J5 pad 06: unconnected-(J5-GND-Pad06) -> GND
- J5 pad 09: unconnected-(J5-GND-Pad09) -> GND
- J5 pad 14: unconnected-(J5-GND-Pad14) -> GND
- J5 pad 20: unconnected-(J5-GND-Pad20) -> GND
- J5 pad 25: unconnected-(J5-GND-Pad25) -> GND
- J5 pad 30: unconnected-(J5-GND-Pad30) -> GND
- J5 pad 34: unconnected-(J5-GND-Pad34) -> GND
- J5 pad 39: unconnected-(J5-GND-Pad39) -> GND

Commit message: PCB update.
Parts:
- added J6: Conn_01x03, Connector_JST:JST_ZH_B3B-ZR_1x03_P1.50mm_Vertical, F.Cu at (39.5, 82.8)
- added J7: Conn_01x03, Connector_JST:JST_ZH_B3B-ZR_1x03_P1.50mm_Vertical, F.Cu at (39.5, 75.0)
- added R1: R_Small_US, Resistor_SMD:R_1206_3216Metric, F.Cu at (69.5, 78.5)
- added R2: R_Small_US, Resistor_SMD:R_1206_3216Metric, F.Cu at (83.5, 78.5)
- DISP1: footprint Displays:TFT LCD - 2.4 - 240x320 -> displays:TFT LCD - 2.4 - 240x320
- moved J5 93.5 mm to (47.5, 89.2), turned to 90 degrees
- moved J3 86.5 mm to (54.1, 89.2), turned to 90 degrees
- moved J1 85.6 mm to (109.2, 88.0)
- moved J4 81.0 mm to (60.8, 89.2), turned to 90 degrees
- moved R3 64.4 mm to (54.2, 78.5), turned to -90 degrees
- moved R4 60.8 mm to (60.8, 78.5), turned to -90 degrees
- moved SW2 37.0 mm to (83.5, 85.2), turned to 0 degrees
- moved SW1 13.3 mm to (69.5, 85.2), turned to 0 degrees
- moved MOD1 2.34 mm to (95.2, 54.8)
- moved DISP1 0.52 mm to (122.0, 82.0)
- renumbered J6 to J1, J5 to J2, J1 to J4, J2 to J5, R2 to R3, R1 to R4
Connections:
- DISP1 pad 1: unconnected-(DISP1-VCC-Pad1) -> +3.3V
- DISP1 pad 2: unconnected-(DISP1-GND-Pad2) -> GND
- DISP1 pad 3: unconnected-(DISP1-CS-Pad3) -> TFT-CS
- DISP1 pad 4: unconnected-(DISP1-RESET-Pad4) -> TFT-RESET
- DISP1 pad 5: unconnected-(DISP1-DC-Pad5) -> TFT-DC
- DISP1 pad 6: unconnected-(DISP1-MOSI-Pad6) -> TFT-MOSI
- DISP1 pad 7: unconnected-(DISP1-SCK-Pad7) -> TFT-SCK
- DISP1 pad 8: unconnected-(DISP1-LED-Pad8) -> +3.3V
- DISP1 pad 9: unconnected-(DISP1-MISO-Pad9) -> TFT-MISO
- J2 pad 08: unconnected-(J5-UART0_TX-Pad08) -> Net-(J2-UART0_TX)
- J2 pad 10: unconnected-(J5-UART0_RX-Pad10) -> Net-(J2-UART0_RX)
- J2 pad 11: unconnected-(J5-GPIO17-Pad11) -> GPIO-0
- J2 pad 13: unconnected-(J5-GPIO27-Pad13) -> GPIO-1
- J3 pad 1: unconnected-(J3-Pin_1-Pad1) -> +5V
- J3 pad 2: unconnected-(J3-Pin_2-Pad2) -> Net-(J3-Pin_2)
- J3 pad 3: unconnected-(J3-Pin_3-Pad3) -> Net-(J3-Pin_3)
- J4 pad 1: unconnected-(J1-Pin_1-Pad1) -> +5V
- J4 pad 2: unconnected-(J1-Pin_2-Pad2) -> Net-(J4-Pin_2)
- J4 pad 3: unconnected-(J1-Pin_3-Pad3) -> Net-(J3-Pin_3)
- J5 pad 1: unconnected-(J2-Pin_1-Pad1) -> +5V
- J5 pad 2: unconnected-(J2-Pin_2-Pad2) -> RC-PWM-0
- J5 pad 3: unconnected-(J2-Pin_3-Pad3) -> Net-(J3-Pin_3)
- MOD1 pad 4: unconnected-(MOD1-SDA-Pad4) -> SDA
- MOD1 pad 5: unconnected-(MOD1-SCL-Pad5) -> SCL
- R3 pad 1: unconnected-(R2-Pad1) -> NEO-0
- R3 pad 2: unconnected-(R2-Pad2) -> Net-(J3-Pin_2)
- R4 pad 1: unconnected-(R1-Pad1) -> NEO-1
- R4 pad 2: unconnected-(R1-Pad2) -> Net-(J4-Pin_2)
- SW1 pad 1: unconnected-(SW1-Pad1) -> BTN-1
- SW1 pad 2: unconnected-(SW1-Pad2) -> GND
- SW2 pad 1: unconnected-(SW2-Pad1) -> BTN-2
- SW2 pad 2: unconnected-(SW2-Pad2) -> GND
- U1 pad 1: unconnected-(U1-PB12-Pad1) -> GPIO-0
- U1 pad 14: unconnected-(U1-PB6-Pad14) -> SCL
- U1 pad 15: unconnected-(U1-PB7-Pad15) -> SDA
- U1 pad 16: unconnected-(U1-PB8-Pad16) -> NEO-0
- U1 pad 17: unconnected-(U1-PB9-Pad17) -> NEO-1
- U1 pad 19: unconnected-(U1-GND-Pad19) -> GND
- U1 pad 2: unconnected-(U1-PB13-Pad2) -> GPIO-1
- U1 pad 26: unconnected-(U1-PA0-Pad26) -> ADC-0
- U1 pad 3: unconnected-(U1-PB14-Pad3) -> GPIO-2
- U1 pad 31: unconnected-(U1-PA5-Pad31) -> TFT-SCK
- U1 pad 32: unconnected-(U1-PA6-Pad32) -> TFT-MISO
- U1 pad 33: unconnected-(U1-PA7-Pad33) -> TFT-MOSI
- U1 pad 34: unconnected-(U1-PB0-Pad34) -> TFT-DC
- U1 pad 35: unconnected-(U1-PB1-Pad35) -> TFT-RESET
- U1 pad 36: unconnected-(U1-PB2-Pad36) -> TFT-CS
- U1 pad 38: unconnected-(U1-3V3-Pad38) -> +3.3V
- U1 pad 39: unconnected-(U1-GND-Pad39) -> GND
- U1 pad 40: unconnected-(U1-5V-Pad40) -> +5V
- U1 pad 5: unconnected-(U1-PA8-Pad5) -> RC-PWM-0
- U1 pad 6: unconnected-(U1-PA9-Pad6) -> Net-(J2-UART0_RX)
- U1 pad 7: unconnected-(U1-PA10-Pad7) -> Net-(J2-UART0_TX)
Other:
- board text added: "5V+"
- board text added: "ADC"
- board text added: "AUX"
- board text added: "BTN0"
- board text added: "BTN1"
- board text added: "GND"
- board text added: "NEO0"
- board text added: "NEO1"
- board text added: "SRV"
