File: pcbs/power_distribution/aux-board/aux-board.kicad_pcb (KiCad board)
At the start: 2 copper layers, 85 x 56 mm, 8 parts, among them J5 Raspberry Pi - Hat Template -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, SW1 SW_Push, SW2 SW_Push, U1 YAAJ_WeAct_BlackPill_Part_Like

Commit message: PCB update.
Parts:
- added J1: Conn_01x02, TerminalBlock_Phoenix:TerminalBlock_Phoenix_PT-1,5-2-5.0-H_1x02_P5.00mm_Horizontal, F.Cu at (109.2, 88.0)
- added J3: Conn_01x03, Connector_JST:JST_ZH_B3B-ZR_1x03_P1.50mm_Vertical, F.Cu at (54.1, 89.2)
- added J4: Conn_01x03, Connector_JST:JST_ZH_B3B-ZR_1x03_P1.50mm_Vertical, F.Cu at (60.8, 89.2)
- added J5: Conn_01x03, Connector_JST:JST_ZH_B3B-ZR_1x03_P1.50mm_Vertical, F.Cu at (47.5, 89.2)
- added J6: Conn_01x03, Connector_JST:JST_ZH_B3B-ZR_1x03_P1.50mm_Vertical, F.Cu at (39.5, 82.8)
- added J7: Conn_01x03, Connector_JST:JST_ZH_B3B-ZR_1x03_P1.50mm_Vertical, F.Cu at (39.5, 75.0)
- added R1: R_Small_US, Resistor_SMD:R_1206_3216Metric, F.Cu at (69.5, 78.5)
- added R2: R_Small_US, Resistor_SMD:R_1206_3216Metric, F.Cu at (83.5, 78.5)
- DISP1: footprint Displays:TFT LCD - 2.4 - 240x320 -> displays:TFT LCD - 2.4 - 240x320
- moved R3 64.4 mm to (54.2, 78.5), turned to -90 degrees
- moved R4 60.8 mm to (60.8, 78.5), turned to -90 degrees
- moved SW2 37.0 mm to (83.5, 85.2), turned to 0 degrees
- moved MOD1 20.8 mm to (95.2, 54.8), turned to -90 degrees
- moved SW1 13.3 mm to (69.5, 85.2), turned to 0 degrees
- moved DISP1 0.52 mm to (122.0, 82.0)
- renumbered J5 to J2, R2 to R3, R1 to R4
Connections:
- DISP1 pad 1: unconnected-(DISP1-VCC-Pad1) -> +3.3V
- DISP1 pad 2: unconnected-(DISP1-GND-Pad2) -> GND
- DISP1 pad 3: unconnected-(DISP1-CS-Pad3) -> TFT-CS
- DISP1 pad 4: unconnected-(DISP1-RESET-Pad4) -> TFT-RESET
- DISP1 pad 5: unconnected-(DISP1-DC-Pad5) -> TFT-DC
- DISP1 pad 6: unconnected-(DISP1-MOSI-Pad6) -> TFT-MOSI
- DISP1 pad 7: unconnected-(DISP1-SCK-Pad7) -> TFT-SCK
- DISP1 pad 8: unconnected-(DISP1-LED-Pad8) -> +3.3V
- DISP1 pad 9: unconnected-(DISP1-MISO-Pad9) -> TFT-MISO
- J2 pad 02: unconnected-(J5-5V_PWR-Pad02) -> +5V
- J2 pad 04: unconnected-(J5-5V_PWR-Pad04) -> +5V
- J2 pad 06: unconnected-(J5-GND-Pad06) -> GND
- J2 pad 08: unconnected-(J5-UART0_TX-Pad08) -> Net-(J2-UART0_TX)
- J2 pad 09: unconnected-(J5-GND-Pad09) -> GND
- J2 pad 10: unconnected-(J5-UART0_RX-Pad10) -> Net-(J2-UART0_RX)
- J2 pad 11: unconnected-(J5-GPIO17-Pad11) -> GPIO-0
- J2 pad 13: unconnected-(J5-GPIO27-Pad13) -> GPIO-1
- J2 pad 14: unconnected-(J5-GND-Pad14) -> GND
- J2 pad 20: unconnected-(J5-GND-Pad20) -> GND
- J2 pad 25: unconnected-(J5-GND-Pad25) -> GND
- J2 pad 30: unconnected-(J5-GND-Pad30) -> GND
- J2 pad 34: unconnected-(J5-GND-Pad34) -> GND
- J2 pad 39: unconnected-(J5-GND-Pad39) -> GND
- MOD1 pad 4: unconnected-(MOD1-SDA-Pad4) -> SDA
- MOD1 pad 5: unconnected-(MOD1-SCL-Pad5) -> SCL
- R3 pad 1: unconnected-(R2-Pad1) -> NEO-0
- R3 pad 2: unconnected-(R2-Pad2) -> Net-(J3-Pin_2)
- R4 pad 1: unconnected-(R1-Pad1) -> NEO-1
- R4 pad 2: unconnected-(R1-Pad2) -> Net-(J4-Pin_2)
- SW1 pad 1: unconnected-(SW1-Pad1) -> BTN-1
- SW1 pad 2: unconnected-(SW1-Pad2) -> GND
- SW2 pad 1: unconnected-(SW2-Pad1) -> BTN-2
- SW2 pad 2: unconnected-(SW2-Pad2) -> GND
- U1 pad 1: unconnected-(U1-PB12-Pad1) -> GPIO-0
- U1 pad 14: unconnected-(U1-PB6-Pad14) -> SCL
- U1 pad 15: unconnected-(U1-PB7-Pad15) -> SDA
- U1 pad 16: unconnected-(U1-PB8-Pad16) -> NEO-0
- U1 pad 17: unconnected-(U1-PB9-Pad17) -> NEO-1
- U1 pad 19: unconnected-(U1-GND-Pad19) -> GND
- U1 pad 2: unconnected-(U1-PB13-Pad2) -> GPIO-1
- U1 pad 26: unconnected-(U1-PA0-Pad26) -> ADC-0
- U1 pad 3: unconnected-(U1-PB14-Pad3) -> GPIO-2
- U1 pad 31: unconnected-(U1-PA5-Pad31) -> TFT-SCK
- U1 pad 32: unconnected-(U1-PA6-Pad32) -> TFT-MISO
- U1 pad 33: unconnected-(U1-PA7-Pad33) -> TFT-MOSI
- U1 pad 34: unconnected-(U1-PB0-Pad34) -> TFT-DC
- U1 pad 35: unconnected-(U1-PB1-Pad35) -> TFT-RESET
- U1 pad 36: unconnected-(U1-PB2-Pad36) -> TFT-CS
- U1 pad 38: unconnected-(U1-3V3-Pad38) -> +3.3V
- U1 pad 39: unconnected-(U1-GND-Pad39) -> GND
- U1 pad 40: unconnected-(U1-5V-Pad40) -> +5V
- U1 pad 5: unconnected-(U1-PA8-Pad5) -> RC-PWM-0
- U1 pad 6: unconnected-(U1-PA9-Pad6) -> Net-(J2-UART0_RX)
- U1 pad 7: unconnected-(U1-PA10-Pad7) -> Net-(J2-UART0_TX)
Other:
- board text added: "5V+"
- board text added: "ADC"
- board text added: "AUX"
- board text added: "BTN0"
- board text added: "BTN1"
- board text added: "GND"
- board text added: "NEO0"
- board text added: "NEO1"
- board text added: "SRV"

Commit message: PCB update.
Parts:
- added J8: Conn_01x04, Connector_PinHeader_2.54mm:PinHeader_1x04_P2.54mm_Horizontal, F.Cu at (71.0, 76.6)
- added J9: Conn_01x05, Connector_PinHeader_2.54mm:PinHeader_1x05_P2.54mm_Horizontal, F.Cu at (105.4, 50.5)
- moved MOD1 27.1 mm to (113.8, 74.6), turned to 90 degrees
- moved R1 9.25 mm to (78.8, 78.8)
- moved SW1 7.60 mm to (75.0, 90.5), turned to 90 degrees
- moved SW2 6.10 mm to (87.0, 90.2), turned to 90 degrees
- moved R4 2.50 mm to (58.2, 78.5)
- moved J4 2.25 mm to (58.5, 89.2)
- moved J1 2.00 mm to (107.2, 88.0)
- moved R3 1.75 mm to (52.5, 78.5)
- moved J3 1.60 mm to (52.5, 89.2)
- moved R2 1.00 mm to (84.5, 78.5)
- moved J5 0.95 mm to (46.5, 89.2)
Connections:
- J2 pad 12: unconnected-(J2-GPIO18-Pad12) -> BCK
- J2 pad 35: unconnected-(J2-GPIO19-Pad35) -> LRCK
- J2 pad 40: unconnected-(J2-GPIO21-Pad40) -> DIN
- J3 pad 3: Net-(J3-Pin_3) -> GND
- J4 pad 3: Net-(J3-Pin_3) -> GND
- J5 pad 3: Net-(J3-Pin_3) -> GND
- J6 pad 2: ADC-1 -> ADC-0
- J7 pad 3: Net-(J3-Pin_3) -> GND
- U1 pad 11: unconnected-(U1-PB3-Pad11) -> NEO-0
- U1 pad 12: unconnected-(U1-PB4-Pad12) -> NEO-1
- U1 pad 16: NEO-0 -> BTN-1
- U1 pad 17: NEO-1 -> BTN-2
- U1 pad 27: unconnected-(U1-PA1-Pad27) -> RC-PWM-0
- U1 pad 5: RC-PWM-0 -> unconnected-(U1-PA8-Pad5)
Routing:
- net +3.3V: track 0.00 -> 207.2 mm, vias 0 -> 6
- net +5V: track 0.00 -> 152.8 mm, vias 0 -> 4
- net TFT-MISO: track 0.00 -> 118.2 mm, vias 0 -> 2
- net TFT-SCK: track 0.00 -> 112.9 mm
- net TFT-MOSI: track 0.00 -> 102.5 mm
- net TFT-DC: track 0.00 -> 96.3 mm
- net TFT-RESET: track 0.00 -> 88.1 mm
- net TFT-CS: track 0.00 -> 83.2 mm
- net ADC-0: track 0.00 -> 58.6 mm
- net RC-PWM-0: track 0.00 -> 55.5 mm
- net SCL: track 0.00 -> 55.3 mm
- net BCK: track 0.00 -> 53.7 mm
- net SDA: track 0.00 -> 53.4 mm
- net Net-(J2-UART0_RX): track 0.00 -> 39.4 mm, vias 0 -> 1
- net Net-(J2-UART0_TX): track 0.00 -> 37.8 mm, vias 0 -> 1
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- added copper zone on B.Cu, net GND
Other:
- board text added: "BNO055 9-DOF SENSOR"
- board text added: "DAC"
- board text added: "ElectroPup Auxiliary Hat metaphasiclabs.com 09/2024"
- board text added: "I2C"
- board text added: "STM32 Bluepill/Blackpill"
