File: pcbs/power_distribution/aux-board/aux-board.kicad_sch (KiCad schematic)
At the start: 6 parts, among them J1 Conn_01x03, J2 Conn_01x03, J3 Conn_01x03, J4 Conn_01x08, J5 Conn_01x06

Commit message: PCB update
Parts:
- removed J5: Conn_01x06, symbol Connector_Generic:Conn_01x06
- added J5: Raspberry Pi - Hat Template - Full Size, General:Raspberry Pi - Hat Template - Full Size, symbol Connectors:Raspberry Pi - Hat Template - Full Size
- added J6: Conn_01x02, symbol Connector_Generic:Conn_01x02
- added R1, R2: R_Small_US, Resistor_SMD:R_1206_3216Metric, symbol Device:R_Small_US
- added SW1, SW2: SW_Push, Button_Switch_THT:SW_PUSH_6mm_H4.3mm, symbol Switch:SW_Push
- added U1: YAAJ_WeAct_BlackPill_Part_Like, MCU_Modules:YAAJ_WeAct_BlackPill_2, symbol MCU_Modules:YAAJ_WeAct_BlackPill_Part_Like
Connections:
- net +5V: now reaches MOD1.1 (Vin)
- net +5V: now also J6.1 (Pin_1)
- net GND: now reaches MOD1.3 (GND)
- net GND: now also J6.2 (Pin_2)
Other:
- note added: "5vDC Power In Isolated DC-DC"
- note removed: "Power In Comms Interface"
- moved on the sheet: J1, J2, J3, J4, MOD1

Commit message: PCB update.
Parts:
- removed J4: Conn_01x08, symbol Connector_Generic:Conn_01x08
- added DISP1: ~, Displays:TFT LCD - 2.4 - 240x320, symbol Displays:TFT_LCD_-_2.4_-_240x320
- added J4: Conn_01x03, Connector_JST:JST_ZH_B3B-ZR_1x03_P1.50mm_Vertical, symbol Connector_Generic:Conn_01x03
- added R3, R5: R_Small_US, Resistor_SMD:R_1206_3216Metric, symbol Device:R_Small_US
- J1, J2, J3: footprint (none) -> Connector_JST:JST_ZH_B3B-ZR_1x03_P1.50mm_Vertical
- J6: footprint (none) -> TerminalBlock_Phoenix:TerminalBlock_Phoenix_PT-1,5-2-5.0-H_1x02_P5.00mm_Horizontal
Connections:
- net +5V: now also J1.1 (Pin_1), J2.1 (Pin_1), J3.1 (Pin_1), J5.02 (5V_PWR), J5.04 (5V_PWR), U1.40 (5V)
- net GND: now also J5.06 (GND), J5.09 (GND), J5.14 (GND), J5.20 (GND), J5.25 (GND), J5.30 (GND), J5.34 (GND), J5.39 (GND), SW1.2, SW2.2, U1.19 (GND), U1.39 (GND), DISP1.2 (GND), J4.3 (Pin_3)
- net at J5.08 (UART0_TX): now also U1.7 (PA10)
- net at J5.10 (UART0_RX): now also U1.6 (PA9)
- net GPIO-0: now reaches J5.11 (GPIO17)
- net GPIO-0: now also U1.1 (PB12)
- net GPIO-1: now reaches J5.13 (GPIO27)
- net GPIO-1: now also U1.2 (PB13)
- net RC-PWM-0: now reaches J2.2 (Pin_2)
- net RC-PWM-0: now also U1.5 (PA8)
- net at J2.3 (Pin_3): now also J1.3 (Pin_3), J3.3 (Pin_3)
- net SDA: now reaches MOD1.4 (SDA)
- net SDA: now also U1.15 (PB7)
- net SCL: now reaches MOD1.5 (SCL)
- net SCL: now also U1.14 (PB6)
- net NEO-0: now reaches R2.1
- net NEO-0: now also U1.16 (PB8)
- net at R2.2: now also J3.2 (Pin_2)
- net BTN-1: now reaches SW1.1
- net BTN-1: now also R3.1
- net at J1.2 (Pin_2): now also R1.2
- net NEO-1: now reaches R1.1
- net NEO-1: now also U1.17 (PB9)
- net ADC-0: now reaches U1.26 (PA0)
- net TFT-SCK: now reaches U1.31 (PA5)
- net TFT-SCK: now also DISP1.7 (SCK)
- net TFT-MISO: now reaches U1.32 (PA6)
- net TFT-MISO: now also DISP1.9 (MISO)
- net TFT-MOSI: now reaches U1.33 (PA7)
- net TFT-MOSI: now also DISP1.6 (MOSI)
- net TFT-DC: now reaches U1.34 (PB0)
- net TFT-DC: now also DISP1.5 (DC)
- net TFT-RESET: now reaches U1.35 (PB1)
- net TFT-RESET: now also DISP1.4 (RESET)
- net TFT-CS: now reaches U1.36 (PB2)
- net TFT-CS: now also DISP1.3 (CS)
- net +3.3V: now reaches U1.38 (3V3)
- net +3.3V: now also DISP1.1 (VCC), DISP1.8 (LED), J4.1 (Pin_1), R3.2, R5.2
- net BTN-2: now reaches SW2.1
- net BTN-2: now also R5.1
- new net ADC-1: J4.2 (Pin_2)
- no-connect marks 0 -> 8
Other:
- note added: "ADC"
- note added: "Buttons"
- note removed: "Button"
- note removed: "LCD Display"
- moved on the sheet: J3, J6, MOD1, R1, R2, SW1, SW2

Commit message: PCB update.
Parts:
- removed DISP1: ~, Displays:TFT LCD - 2.4 - 240x320, symbol Displays:TFT_LCD_-_2.4_-_240x320
- added DISP1: ~, displays:TFT LCD - 2.4 - 240x320, symbol displays:TFT_LCD_-_2.4_-_240x320
- added J7: Conn_01x03, Connector_JST:JST_ZH_B3B-ZR_1x03_P1.50mm_Vertical, symbol Connector_Generic:Conn_01x03
- renumbered J6 to J1, J5 to J2, J1 to J4, J2 to J5, J4 to J6, R3 to R1, R5 to R2, R2 to R3, R1 to R4
Connections:
- net +3.3V: now also DISP1.1 (VCC), DISP1.8 (LED)
- net +5V: now also J7.1 (Pin_1)
- net GND: now also DISP1.2 (GND)
- net TFT-CS: now also DISP1.3 (CS)
- net TFT-DC: now also DISP1.5 (DC)
- net TFT-MISO: now also DISP1.9 (MISO)
- net TFT-MOSI: now also DISP1.6 (MOSI)
- net TFT-RESET: now also DISP1.4 (RESET)
- net TFT-SCK: now also DISP1.7 (SCK)
- net at J3.3 (Pin_3), J4.3 (Pin_3), J5.3 (Pin_3): now also J7.3 (Pin_3)
- net GPIO-2: now reaches U1.3 (PB14)
- net GPIO-2: now also J7.2 (Pin_2)
Other:
- note added: "AUX"
- moved on the sheet: J3, J4, J5, J6, R3, R4

Commit message: PCB update.
Parts:
- added J8: Conn_01x04, Connector_PinHeader_2.54mm:PinHeader_1x04_P2.54mm_Horizontal, symbol Connector_Generic:Conn_01x04
- added J9: Conn_01x05, Connector_PinHeader_2.54mm:PinHeader_1x05_P2.54mm_Horizontal, symbol Connector_Generic:Conn_01x05
Connections:
- net ADC-1 is gone; now on net ADC-0: J6.2 (Pin_2)
- net +3.3V: now also J8.1 (Pin_1), J9.5 (Pin_5)
- net BTN-1: now also U1.16 (PB8)
- net BTN-2: now also U1.17 (PB9)
- net GND: now also J3.3 (Pin_3), J4.3 (Pin_3), J5.3 (Pin_3), J7.3 (Pin_3), J8.4 (Pin_4), J9.4 (Pin_4)
- net NEO-0: now also U1.11 (PB3); no longer U1.16 (PB8)
- net NEO-1: now also U1.12 (PB4); no longer U1.17 (PB9)
- net RC-PWM-0: now also U1.27 (PA1); no longer U1.5 (PA8)
- net SCL: now also J8.3 (Pin_3)
- net SDA: now also J8.2 (Pin_2)
- net BCK: now reaches J2.12 (GPIO18)
- net BCK: now also J9.1 (Pin_1)
- net LRCK: now reaches J2.35 (GPIO19)
- net LRCK: now also J9.3 (Pin_3)
- net DIN: now reaches J2.40 (GPIO21)
- net DIN: now also J9.2 (Pin_2)
- no-connect marks 8 -> 49
Other:
- note added: "AUDIO DAC"
- note added: "I2C AUX"
- moved on the sheet: DISP1, J2, J3, J4, J5, J6, J7, R3, R4
