File: pcbs/auxiliary-pi-hat/auxiliary-pi-hat.kicad_pcb (KiCad board)
At the start: 2 copper layers, 85 x 56 mm, 19 parts, among them J1 Conn_01x02, J2 Raspberry Pi - Hat Template -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, J3 Conn_01x03, J4 Conn_01x03, J5 Conn_01x03, J6 Conn_01x03, J7 Conn_01x03, J8 Conn_01x04, J9 Conn_01x05, SW1 SW_Push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

Commit message: aux pcb update
Parts:
- removed J6: Conn_01x03, Connector_JST:JST_ZH_B3B-ZR_1x03_P1.50mm_Vertical
- removed SW2: SW_Push, Button_Switch_THT:SW_PUSH_6mm_H4.3mm
- added J10: Conn_01x03, Connector_JST:JST_ZH_B3B-ZR_1x03_P1.50mm_Vertical, F.Cu at (145.0, 98.5)
- added J11: Conn_01x03, Connector_JST:JST_ZH_B3B-ZR_1x03_P1.50mm_Vertical, F.Cu at (119.4, 98.5)
- added Q1: BSS138, Package_TO_SOT_SMD:SOT-23, F.Cu at (184.5, 94.3)
- added Q2: BSS138, Package_TO_SOT_SMD:SOT-23, F.Cu at (186.5, 83.5)
- added R5: 10k, Resistor_SMD:R_1206_3216Metric, F.Cu at (187.5, 59.8)
- added R6: 10k, Resistor_SMD:R_1206_3216Metric, F.Cu at (186.9, 65.0)
- added R7: 10k, Resistor_SMD:R_1206_3216Metric, F.Cu at (186.9, 68.2)
- added R8: 10k, Resistor_SMD:R_1206_3216Metric, F.Cu at (186.9, 71.5)
- added R9: 500, Resistor_SMD:R_1206_3216Metric, F.Cu at (186.9, 74.8)
- added U2: SN74LVC1G14DBV, Package_TO_SOT_SMD:SOT-23-5, F.Cu at (129.0, 108.5)
- DISP1: footprint displays:TFT LCD - 2.4 - 240x320 -> displays:LCD-Display-1.8-128x160-Hiletgo
- J7: value Conn_01x03 -> Conn_01x04; footprint Connector_JST:JST_ZH_B3B-ZR_1x03_P1.50mm_Vertical -> Connector_JST:JST_ZH_B4B-ZR_1x04_P1.50mm_Vertical
- J8: value Conn_01x04 -> Conn_02x04_Odd_Even; footprint Connector_PinHeader_2.54mm:PinHeader_1x04_P2.54mm_Horizontal -> Connector_PinHeader_2.54mm:PinHeader_2x04_P2.54mm_Vertical
- J9: footprint Connector_PinHeader_2.54mm:PinHeader_1x05_P2.54mm_Horizontal -> Connector_JST:JST_ZH_B5B-ZR_1x05_P1.50mm_Vertical
- R3: value R_Small_US -> 500
- moved G*** 165.9 mm to (239.5, 133.0)
- moved J8 101.1 mm to (168.8, 50.7)
- moved R3 91.3 mm to (139.8, 110.2)
- moved R4 91.3 mm to (144.0, 110.0)
- moved SW1 87.6 mm to (162.5, 95.0), turned to 0 degrees
- moved J4 80.6 mm to (138.6, 98.5)
- moved J3 80.2 mm to (132.2, 98.5)
- moved J5 79.8 mm to (125.8, 98.5)
- moved J7 77.2 mm to (113.0, 98.5), turned to 90 degrees
- moved U1 58.2 mm to (95.8, 82.6)
- moved J2 54.7 mm to (123.5, 50.6)
- moved DISP1 54.3 mm to (175.4, 91.9)
- moved R2 48.4 mm to (122.5, 108.5)
- moved R1 47.3 mm to (115.5, 108.5)
- moved MOD1 36.8 mm to (150.1, 68.7), turned to -90 degrees
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Connections:
- net GPIO-0 renamed GPIO-17
- J2 pad 03: unconnected-(J2-GPIO02/SDA1-Pad03) -> SDA
- J2 pad 05: unconnected-(J2-GPIO03/SCL-Pad05) -> SCL
- J2 pad 13: GPIO-1 -> unconnected-(J2-GPIO27-Pad13)
- J2 pad 29: unconnected-(J2-GPIO05-Pad29) -> SBUS
- J2 pad 33: unconnected-(J2-GPIO13-Pad33) -> GPIO-13
- J2 pad 36: unconnected-(J2-GPIO16-Pad36) -> GPIO-16
- J2 pad 37: unconnected-(J2-GPIO26-Pad37) -> GPIO-26
- J2 pad 38: unconnected-(J2-GPIO20-Pad38) -> GPIO-20
- J4 pad 1: +5V -> unconnected-(J4-Pin_1-Pad1)
- J4 pad 2: Net-(J4-Pin_2) -> GPIO-2
- J7 pad 1: +5V -> +3.3V
- J7 pad 2: GPIO-2 -> SDA_MCU
- J7 pad 3: GND -> SCL_MCU
- J8 pad 1: +3.3V -> GPIO-20
- J8 pad 2: SDA -> GND
- J8 pad 3: SCL -> GPIO-16
- R3 pad 1: NEO-0 -> Net-(Q1-D)
- U1 pad 14: SCL -> SCL_MCU
- U1 pad 15: SDA -> SDA_MCU
- U1 pad 17: BTN-2 -> unconnected-(U1-PB9-Pad17)
- U1 pad 2: GPIO-1 -> unconnected-(U1-PB13-Pad2)
- U1 pad 26: ADC-0 -> unconnected-(U1-PA0-Pad26)
- U1 pad 3: GPIO-2 -> unconnected-(U1-PB14-Pad3)
- U1 pad 32: TFT-MISO -> unconnected-(U1-PA6-Pad32)
Routing:
- net +3.3V: track 209.3 -> 0.00 mm, vias 6 -> 0
- net +5V: track 152.8 -> 0.00 mm, vias 4 -> 0
- net TFT-MISO: track 115.7 -> 0.00 mm, vias 2 -> 0
- net TFT-SCK: track 112.9 -> 0.00 mm
- net TFT-MOSI: track 102.5 -> 0.00 mm
- net TFT-DC: track 96.3 -> 0.00 mm
- net TFT-RESET: track 88.1 -> 0.00 mm
- net TFT-CS: track 83.2 -> 0.00 mm
- net ADC-0: track 58.6 -> 0.00 mm
- net SCL: track 55.3 -> 0.00 mm
- net RC-PWM-0: track 54.8 -> 0.00 mm
- net BCK: track 53.7 -> 0.00 mm
- net SDA: track 53.4 -> 0.00 mm
- net Net-(J2-UART0_RX): track 39.4 -> 0.00 mm, vias 1 -> 0
- net Net-(J2-UART0_TX): track 37.8 -> 0.00 mm, vias 1 -> 0
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Other:
- board text removed: "ADC"
