File: pcbs/power_carrier/power_carrier.kicad_pcb (KiCad board)
At the start: 2 copper layers, 74 x 240 mm, 29 parts, among them J1 Conn_01x03, J10 Conn_01x06, J11 Conn_01x06, J12 Conn_01x06, J13 Conn_01x06, J14 Conn_01x06, J15 Conn_01x06, J16 Conn_01x06, J2 Conn_01x03, J20 Conn_01x03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

Commit message: power carrier PCB fix
Connections:
- J3 pad 1: /ISO 5vDC GND -> /ISO 5vDC+
- J3 pad 2: /ISO 5vDC+ -> /ISO 5vDC GND
Routing:
- net /ISO 5vDC+: track 22.3 -> 17.9 mm
Changed lines of the file:
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@@
 		)
 		(sheetname "Root")
-		(sheetfile "power_distribution.kicad_sch")
+		(sheetfile "power_carrier.kicad_sch")
 		(attr through_hole)
 		(fp_rect
@@
 		(property ki_fp_filters "Connector*:*_1x??_*")
 		(sheetname "Root")
-		(sheetfile "power_distribution.kicad_sch")
+		(sheetfile "power_carrier.kicad_sch")
 		(attr through_hole)
 		(fp_line
@@
 		(property ki_fp_filters "Connector*:*_1x??_*")
 		(sheetname "Root")
-		(sheetfile "power_distribution.kicad_sch")
+		(sheetfile "power_carrier.kicad_sch")
 		(attr through_hole)
 		(fp_line
@@
 		)
 		(sheetname "Root")
-		(sheetfile "power_distribution.kicad_sch")
+		(sheetfile "power_carrier.kicad_sch")
 		(attr through_hole)
 		(fp_line
@@
 		(property ki_fp_filters "Connector*:*_1x??_*")
 		(sheetname "Root")
-		(sheetfile "power_distribution.kicad_sch")
+		(sheetfile "power_carrier.kicad_sch")
 		(attr through_hole)
 		(fp_line
@@
 		(property ki_fp_filters "LED* LED_SMD:* LED_THT:*")
 		(sheetname "Root")
-		(sheetfile "power_distribution.kicad_sch")
+		(sheetfile "power_carrier.kicad_sch")
 		(attr smd)
 		(fp_line
@@
 		(property ki_fp_filters "Connector*:*_1x??_*")
 		(sheetname "Root")
-		(sheetfile "power_distribution.kicad_sch")
+		(sheetfile "power_carrier.kicad_sch")
 		(attr through_hole)
 		(fp_line
@@
 		)
 		(sheetname "Root")
-		(sheetfile "power_distribution.kicad_sch")
+		(sheetfile "power_carrier.kicad_sch")
 		(attr through_hole)
 		(fp_line
@@
 		(property ki_fp_filters "Connector*:*_1x??_*")
 		(sheetname "Root")
-		(sheetfile "power_distribution.kicad_sch")
+		(sheetfile "power_carrier.kicad_sch")
 		(attr through_hole)
 		(fp_line
@@
 			(layers "*.Cu" "*.Mask")
 			(remove_unused_layers no)
-			(net 16 "/ISO 5vDC GND")
+			(net 17 "/ISO 5vDC+")
 			(pinfunction "Pin_1")
 			(pintype "passive")
@@
 			(layers "*.Cu" "*.Mask")
 			(remove_unused_layers no)
-			(net 17 "/ISO 5vDC+")
+			(net 16 "/ISO 5vDC GND")
 			(pinfunction "Pin_2")
 			(pintype "passive")
@@
 		(property ki_fp_filters "Connector*:*_1x??_*")
 		(sheetname "Root")
-		(sheetfile "power_distribution.kicad_sch")
+		(sheetfile "power_carrier.kicad_sch")
 		(attr through_hole)
 		(fp_line
@@
 		(property ki_fp_filters "Connector*:*_1x??_*")
 		(sheetname "Root")
-		(sheetfile "power_distribution.kicad_sch")
+		(sheetfile "power_carrier.kicad_sch")
 		(attr through_hole)
 		(fp_line
@@
 		(property ki_fp_filters "Connector*:*_1x??_*")
 		(sheetname "Root")
-		(sheetfile "power_distribution.kicad_sch")
+		(sheetfile "power_carrier.kicad_sch")
 		(attr through_hole)
 		(fp_line
@@
 		(property ki_fp_filters "Connector*:*_1x??_*")
 		(sheetname "Root")
-		(sheetfile "power_distribution.kicad_sch")
+		(sheetfile "power_carrier.kicad_sch")
 		(attr through_hole)
 		(fp_line
@@
 		(property ki_fp_filters "Connector*:*_1x??_*")
 		(sheetname "Root")
-		(sheetfile "power_distribution.kicad_sch")
+		(sheetfile "power_carrier.kicad_sch")
 		(attr through_hole)
 		(fp_line
@@
 		(property ki_fp_filters "Connector*:*_1x??_*")
 		(sheetname "Root")
-		(sheetfile "power_distribution.kicad_sch")
+		(sheetfile "power_carrier.kicad_sch")
 		(attr through_hole)
 		(fp_line
@@
 		(property ki_fp_filters "Connector*:*_1x??_*")
 		(sheetname "Root")
-		(sheetfile "power_distribution.kicad_sch")
+		(sheetfile "power_carrier.kicad_sch")
 		(attr through_hole)
 		(fp_line
@@
 		(property ki_fp_filters "R_*")
 		(sheetname "Root")
-		(sheetfile "power_distribution.kicad_sch")
+		(sheetfile "power_carrier.kicad_sch")
 		(attr smd)
 		(fp_line
@@
 		(property ki_fp_filters "Connector*:*_1x??_*")
 		(sheetname "Root")
-		(sheetfile "power_distribution.kicad_sch")
+		(sheetfile "power_carrier.kicad_sch")
 		(attr through_hole)
 		(fp_line
@@
 		(property ki_fp_filters "Connector*:*_1x??_*")
 		(sheetname "Root")
-		(sheetfile "power_distribution.kicad_sch")
+		(sheetfile "power_carrier.kicad_sch")
 		(attr through_hole)
 		(fp_line
@@
 		(property ki_fp_filters "Connector*:*_1x??_*")
 		(sheetname "Root")
-		(sheetfile "power_distribution.kicad_sch")
+		(sheetfile "power_carrier.kicad_sch")
 		(attr through_hole)
 		(fp_line
@@
 		(property ki_fp_filters "Connector*:*_1x??_*")
 		(sheetname "Root")
-		(sheetfile "power_distribution.kicad_sch")
+		(sheetfile "power_carrier.kicad_sch")
 		(attr through_hole)
 		(fp_line
@@
 		(property ki_fp_filters "Connector*:*_1x??_*")
 		(sheetname "Root")
-		(sheetfile "power_distribution.kicad_sch")
+		(sheetfile "power_carrier.kicad_sch")
 		(attr through_hole)
 		(fp_line
@@
 		)
 		(sheetname "Root")
-		(sheetfile "power_distribution.kicad_sch")
+		(sheetfile "power_carrier.kicad_sch")
 		(fp_rect
 			(start 0 0)
@@
 		(property ki_fp_filters "SolderJumper*Open*")
 		(sheetname "Root")
-		(sheetfile "power_distribution.kicad_sch")
+		(sheetfile "power_carrier.kicad_sch")
 		(zone_connect 1)
 		(attr exclude_from_pos_files exclude_from_bom)
@@
 		(property ki_fp_filters "SolderJumper*Open*")
 		(sheetname "Root")
-		(sheetfile "power_distribution.kicad_sch")
+		(sheetfile "power_carrier.kicad_sch")
 		(zone_connect 1)
 		(attr exclude_from_pos_files exclude_from_bom)
@@
 		(property ki_fp_filters "SolderJumper*Open*")
 		(sheetname "Root")
-		(sheetfile "power_distribution.kicad_sch")
+		(sheetfile "power_carrier.kicad_sch")
 		(zone_connect 1)
 		(attr exclude_from_pos_files exclude_from_bom)
@@
 		(property ki_fp_filters "SolderJumper*Open*")
 		(sheetname "Root")
-		(sheetfile "power_distribution.kicad_sch")
+		(sheetfile "power_carrier.kicad_sch")
 		(zone_connect 1)
 		(attr exclude_from_pos_files exclude_from_bom)
@@
 	)
 	(gr_text "-"
-		(at 201.5 189.5 180)
+		(at 201.25 184.75 180)
 		(layer "F.SilkS")
 		(effects
@@
 	)
 	(gr_text "+\n"
-		(at 201.5 184.5 180)
+		(at 201.5 189.75 180)
 		(layer "F.SilkS")
 		(effects
@@
 	)
 	(segment
-		(start 186 191)
-		(end 192.805 191)
-		(width 3)
-		(layer "F.Cu")
-		(net 16)
-	)
-	(segment
 		(start 181.48 188.26)
-		(end 183.26 188.26)
+		(end 183.74 186)
 		(width 3)
 		(layer "F.Cu")
@@
 	)
 	(segment
-		(start 183.26 188.26)
-		(end 186 191)
+		(start 183.74 186)
+		(end 192.805 186)
 		(width 3)
 		(layer "F.Cu")
@@
 	)
 	(segment
-		(start 176.4 188.26)
-		(end 176.4 185.1)
-		(width 3)
-		(layer "F.Cu")
-		(net 17)
-	)
-	(segment
-		(start 192 183.5)
-		(end 192.805 184.305)
-		(width 3)
-		(layer "F.Cu")
-		(net 17)
-	)
-	(segment
-		(start 176.4 185.1)
-		(end 178 183.5)
+		(start 192.345 191.46)
+		(end 192.805 191)
 		(width 3)
 		(layer "F.Cu")
@@
 	)
 	(segment
-		(start 178 183.5)
-		(end 192 183.5)
+		(start 179.6 191.46)
+		(end 192.345 191.46)
 		(width 3)
 		(layer "F.Cu")
@@
 	)
 	(segment
-		(start 192.805 184.305)
-		(end 192.805 186)
+		(start 176.4 188.26)
+		(end 179.6 191.46)
 		(width 3)
 		(layer "F.Cu")
