File: pcbs/power_carrier/power_carrier.kicad_sch (KiCad schematic)
At the start: 28 parts, among them J1 Conn_01x03, J10 Conn_01x06, J11 Conn_01x06, J12 Conn_01x06, J13 Conn_01x06, J14 Conn_01x06, J15 Conn_01x06, J16 Conn_01x06, J2 Conn_01x03, J20 Conn_01x03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

Commit message: power carrier PCB fix
Connections:
- net ISO 5vDC GND: now also J3.2 (Pin_2), U1.16 (-VOUT); no longer J3.1 (Pin_1), U1.14 (+VOUT)
- net ISO 5vDC+: now also J3.1 (Pin_1), U1.14 (+VOUT); no longer J3.2 (Pin_2), U1.16 (-VOUT)
Changed lines of the file:
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@@
 		)
 	)
-	(label "ISO 5vDC GND"
+	(label "ISO 5vDC+"
 		(at 167.64 53.34 0)
 		(fields_autoplaced yes)
@@
 		)
 	)
-	(label "ISO 5vDC+"
+	(label "ISO 5vDC GND"
 		(at 154.94 55.88 0)
 		(fields_autoplaced yes)
