File: pcbs/auxiliary-board/auxiliary-board.kicad_pcb (KiCad board)
At the start: 2 copper layers, 93 x 56 mm, 33 parts, among them J1 Conn_01x02, J10 Conn_01x03, J11 Conn_01x03, J2 Raspberry Pi - Hat Template -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, J3 Conn_01x03, J4 Conn_01x03, J5 Conn_01x03, J7 Conn_01x04, J8 Conn_02x04_Odd_Even, J9 Conn_01x05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

Commit message: push assets
Other:
- board text added: "ElectroPup Auxiliary Pi Hat metaphasiclabs.com v1.0 : 10/2024"
- board text removed: "ElectroPup Auxiliary Pi Hat metaphasiclabs.com 10/2024"
Changed lines of the file:
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@@
 		(tags "resistor")
 		(property "Reference" "R2"
-			(at -0.0375 2 360)
+			(at -0.0375 2 0)
 			(layer "F.SilkS")
 			(effects
@@
 		)
 		(property "Value" "10k"
-			(at 0 1.82 360)
+			(at 0 1.82 0)
 			(layer "F.Fab")
 			(effects
@@
 		)
 		(fp_text user "${REFERENCE}"
-			(at 0 0 360)
+			(at 0 0 0)
 			(layer "F.Fab")
 			(effects
@@
 		)
 		(property "Value" "YAAJ_WeAct_BlackPill_Part_Like"
-			(at 20.32 24.765 360)
+			(at 20.32 24.765 0)
 			(layer "F.Fab")
 			(hide yes)
@@
 		)
 		(fp_text user "REF**"
-			(at 7.62 24.13 360)
+			(at 7.62 24.13 0)
 			(layer "F.Fab")
 			(effects
@@
 			(pintype "power_in")
 		)
-		(model "D:/Users/admin/Documents/KiCad/Libraries/packages3d/Modules/STM32_Blue_Pill/YAAJ_BluePill_PinHeaders_H_SWD_cp.wrl"
-			(offset
-				(xyz 0 0 0)
-			)
-			(scale
-				(xyz 1 1 1)
-			)
-			(rotate
-				(xyz 0 0 0)
-			)
-		)
-		(model "D:/Users/admin/Documents/KiCad/Libraries/packages3d/Modules/STM32_Blue_Pill/YAAJ_BluePill_PinHeaders_No_SWD_cp.wrl"
-			(offset
-				(xyz 0 0 0)
-			)
-			(scale
-				(xyz 1 1 1)
-			)
-			(rotate
-				(xyz 0 0 0)
-			)
-		)
-		(model "D:/Users/admin/Documents/KiCad/Libraries/packages3d/Modules/STM32_Blue_Pill/YAAJ_BluePill_PinHeaders_V_SWD_cp.wrl"
-			(offset
-				(xyz 0 0 0)
-			)
-			(scale
-				(xyz 1 1 1)
-			)
-			(rotate
-				(xyz 0 0 0)
-			)
-		)
-		(model "D:/Users/admin/Documents/KiCad/Libraries/packages3d/Modules/STM32_Blue_Pill/YAAJ_BluePill_PinSockets_H_SWD_cp.wrl"
-			(offset
-				(xyz 0 0 0)
-			)
-			(scale
-				(xyz 1 1 1)
-			)
-			(rotate
-				(xyz 0 0 0)
-			)
-		)
-		(model "D:/Users/admin/Documents/KiCad/Libraries/packages3d/Modules/STM32_Blue_Pill/YAAJ_BluePill_PinSockets_No_SWD_cp.wrl"
+		(model "/home/pc/Desktop/projects/kicad-libraries/mcus/mcus.pretty/3dmodels/blackpill v2.0.step"
 			(offset
-				(xyz 0 0 0)
+				(xyz 7.6 -25 0)
 			)
 			(scale
@@
 			)
 			(rotate
-				(xyz 0 0 0)
-			)
-		)
-		(model "D:/Users/admin/Documents/KiCad/Libraries/packages3d/Modules/STM32_Blue_Pill/YAAJ_BluePill_PinSockets_V_SWD_cp.wrl"
-			(offset
-				(xyz 0 0 0)
-			)
-			(scale
-				(xyz 1 1 1)
-			)
-			(rotate
-				(xyz 0 0 0)
+				(xyz 0 0 90)
 			)
 		)
@@
 		(tags "connector JST ZH vertical")
 		(property "Reference" "J11"
-			(at 1.5 -2.5 360)
+			(at 1.5 -2.5 0)
 			(layer "F.SilkS")
 			(effects
@@
 		)
 		(property "Value" "Conn_01x03"
-			(at 1.5 3.4 360)
+			(at 1.5 3.4 0)
 			(layer "F.Fab")
 			(effects
@@
 		)
 		(property "Footprint" "Connector_JST:JST_ZH_B3B-ZR_1x03_P1.50mm_Vertical"
-			(at 0 0 360)
+			(at 0 0 0)
 			(layer "F.Fab")
 			(hide yes)
@@
 		)
 		(property "Datasheet" ""
-			(at 0 0 360)
+			(at 0 0 0)
 			(layer "F.Fab")
 			(hide yes)
@@
 		)
 		(property "Description" "Generic connector, single row, 01x03, script generated (kicad-library-utils/schlib/autogen/connector/)"
-			(at 0 0 360)
+			(at 0 0 0)
 			(layer "F.Fab")
 			(hide yes)
@@
 		)
 		(fp_text user "${REFERENCE}"
-			(at 1.5 1.5 360)
+			(at 1.5 1.5 0)
 			(layer "F.Fab")
 			(effects
@@
 		(tags "tact sw push 6mm")
 		(property "Reference" "SW1"
-			(at 3.25 2.25 360)
+			(at 3.25 2.25 0)
 			(layer "F.SilkS")
 			(effects
@@
 		(tags "resistor")
 		(property "Reference" "R1"
-			(at 1.25 1.75 360)
+			(at 1.25 1.75 0)
 			(layer "F.SilkS")
 			(effects
@@
 		)
 		(property "Value" "R_Small_US"
-			(at 0 1.82 360)
+			(at 0 1.82 0)
 			(layer "F.Fab")
 			(hide yes)
@@
 		)
 		(fp_text user "${REFERENCE}"
-			(at 0 0 360)
+			(at 0 0 0)
 			(layer "F.Fab")
 			(effects
@@
 		)
 		(fp_text user "${REFERENCE}"
-			(at 1.27 3.81 360)
+			(at 1.27 3.81 0)
 			(layer "F.Fab")
 			(effects
@@
 		(at 97.25 75.5 180)
 		(property "Reference" "G***"
-			(at 3.5 7.25 360)
+			(at 3.5 7.25 0)
 			(layer "B.SilkS")
 			(hide yes)
@@
 		)
 		(property "Value" "LOGO"
-			(at -1.5 8 360)
+			(at -1.5 8 0)
 			(layer "B.SilkS")
 			(hide yes)
@@
 		)
 		(property "Footprint" "graphics:electroPup-graphic-20mm"
-			(at 0 0 360)
+			(at 0 0 0)
 			(layer "B.Fab")
 			(hide yes)
@@
 		)
 		(property "Datasheet" ""
-			(at 0 0 360)
+			(at 0 0 0)
 			(layer "B.Fab")
 			(hide yes)
@@
 		)
 		(property "Description" ""
-			(at 0 0 360)
+			(at 0 0 0)
 			(layer "B.Fab")
 			(hide yes)
@@
 		)
 	)
-	(gr_text "ElectroPup\nAuxiliary Pi Hat\nmetaphasiclabs.com\n10/2024"
+	(gr_text "ElectroPup\nAuxiliary Pi Hat\nmetaphasiclabs.com\nv1.0 : 10/2024"
 		(at 133.5 80.25 0)
 		(layer "B.SilkS")

Commit message: cleanup
Connections:
- MOD1 pad 4: SDA -> SCL
- MOD1 pad 5: SCL -> SDA
Routing:
- net SCL: track 65.6 -> 71.1 mm
- net SDA: track 65.7 -> 67.5 mm
Other:
- board text added: "ElectroPup Auxiliary Pi Hat metaphasiclabs.com v1.1 : 10/2024"
- board text removed: "ElectroPup Auxiliary Pi Hat metaphasiclabs.com v1.0 : 10/2024"
Changed lines of the file:
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@@
 		(property ki_fp_filters "R_*")
 		(sheetname "Root")
-		(sheetfile "auxiliary-pi-hat.kicad_sch")
+		(sheetfile "auxiliary-board.kicad_sch")
 		(attr smd)
 		(fp_line
@@
 		(property ki_fp_filters "R_*")
 		(sheetname "Root")
-		(sheetfile "auxiliary-pi-hat.kicad_sch")
+		(sheetfile "auxiliary-board.kicad_sch")
 		(attr smd)
 		(fp_line
@@
 		(property ki_fp_filters "SOT?23*")
 		(sheetname "Root")
-		(sheetfile "auxiliary-pi-hat.kicad_sch")
+		(sheetfile "auxiliary-board.kicad_sch")
 		(attr smd)
 		(fp_line
@@
 		(property ki_fp_filters "R_*")
 		(sheetname "Root")
-		(sheetfile "auxiliary-pi-hat.kicad_sch")
+		(sheetfile "auxiliary-board.kicad_sch")
 		(attr smd)
 		(fp_line
@@
 		(property ki_fp_filters "R_*")
 		(sheetname "Root")
-		(sheetfile "auxiliary-pi-hat.kicad_sch")
+		(sheetfile "auxiliary-board.kicad_sch")
 		(attr smd)
 		(fp_line
@@
 		)
 		(sheetname "Root")
-		(sheetfile "auxiliary-pi-hat.kicad_sch")
+		(sheetfile "auxiliary-board.kicad_sch")
 		(attr through_hole)
 		(fp_line
@@
 		(property ki_fp_filters "R_*")
 		(sheetname "Root")
-		(sheetfile "auxiliary-pi-hat.kicad_sch")
+		(sheetfile "auxiliary-board.kicad_sch")
 		(attr smd)
 		(fp_line
@@
 		(property ki_fp_filters "R_*")
 		(sheetname "Root")
-		(sheetfile "auxiliary-pi-hat.kicad_sch")
+		(sheetfile "auxiliary-board.kicad_sch")
 		(attr smd)
 		(fp_line
@@
 		(property ki_fp_filters "R_*")
 		(sheetname "Root")
-		(sheetfile "auxiliary-pi-hat.kicad_sch")
+		(sheetfile "auxiliary-board.kicad_sch")
 		(attr smd)
 		(fp_line
@@
 		(property ki_fp_filters "Connector*:*_1x??_*")
 		(sheetname "Root")
-		(sheetfile "auxiliary-pi-hat.kicad_sch")
+		(sheetfile "auxiliary-board.kicad_sch")
 		(attr through_hole)
 		(fp_line
@@
 		)
 		(sheetname "Root")
-		(sheetfile "auxiliary-pi-hat.kicad_sch")
+		(sheetfile "auxiliary-board.kicad_sch")
 		(attr through_hole)
 		(fp_line
@@
 		(property ki_fp_filters "SOT?23*")
 		(sheetname "Root")
-		(sheetfile "auxiliary-pi-hat.kicad_sch")
+		(sheetfile "auxiliary-board.kicad_sch")
 		(attr smd)
 		(fp_line
@@
 		(property ki_fp_filters "R_*")
 		(sheetname "Root")
-		(sheetfile "auxiliary-pi-hat.kicad_sch")
+		(sheetfile "auxiliary-board.kicad_sch")
 		(attr smd)
 		(fp_line
@@
 		(property ki_fp_filters "Connector*:*_1x??_*")
 		(sheetname "Root")
-		(sheetfile "auxiliary-pi-hat.kicad_sch")
+		(sheetfile "auxiliary-board.kicad_sch")
 		(attr through_hole)
 		(fp_line
@@
 		(property ki_fp_filters "Connector*:*_1x??_*")
 		(sheetname "Root")
-		(sheetfile "auxiliary-pi-hat.kicad_sch")
+		(sheetfile "auxiliary-board.kicad_sch")
 		(attr through_hole)
 		(fp_line
@@
 		(property ki_fp_filters "SOT*23*")
 		(sheetname "Root")
-		(sheetfile "auxiliary-pi-hat.kicad_sch")
+		(sheetfile "auxiliary-board.kicad_sch")
 		(attr smd)
 		(fp_line
@@
 		(property ki_fp_filters "Connector*:*_1x??_*")
 		(sheetname "Root")
-		(sheetfile "auxiliary-pi-hat.kicad_sch")
+		(sheetfile "auxiliary-board.kicad_sch")
 		(attr through_hole)
 		(fp_line
@@
 		)
 		(sheetname "Root")
-		(sheetfile "auxiliary-pi-hat.kicad_sch")
+		(sheetfile "auxiliary-board.kicad_sch")
 		(attr through_hole)
 		(fp_line
@@
 		(property ki_fp_filters "Connector*:*_1x??_*")
 		(sheetname "Root")
-		(sheetfile "auxiliary-pi-hat.kicad_sch")
+		(sheetfile "auxiliary-board.kicad_sch")
 		(attr through_hole)
 		(fp_line
@@
 		(property ki_fp_filters "R_*")
 		(sheetname "Root")
-		(sheetfile "auxiliary-pi-hat.kicad_sch")
+		(sheetfile "auxiliary-board.kicad_sch")
 		(attr smd)
 		(fp_line
@@
 		)
 		(sheetname "Root")
-		(sheetfile "auxiliary-pi-hat.kicad_sch")
+		(sheetfile "auxiliary-board.kicad_sch")
 		(attr through_hole)
 		(fp_rect
@@
 		(property ki_fp_filters "Connector*:*_1x??_*")
 		(sheetname "Root")
-		(sheetfile "auxiliary-pi-hat.kicad_sch")
+		(sheetfile "auxiliary-board.kicad_sch")
 		(attr through_hole)
 		(fp_line
@@
 		(property ki_fp_filters "Connector*:*_2x??_*")
 		(sheetname "Root")
-		(sheetfile "auxiliary-pi-hat.kicad_sch")
+		(sheetfile "auxiliary-board.kicad_sch")
 		(attr through_hole)
 		(fp_line
@@
 		)
 		(sheetname "Root")
-		(sheetfile "auxiliary-pi-hat.kicad_sch")
+		(sheetfile "auxiliary-board.kicad_sch")
 		(attr through_hole)
 		(fp_line
@@
 		(property ki_fp_filters "R_*")
 		(sheetname "Root")
-		(sheetfile "auxiliary-pi-hat.kicad_sch")
+		(sheetfile "auxiliary-board.kicad_sch")
 		(attr smd)
 		(fp_line
@@
 		(property ki_fp_filters "Connector*:*_1x??_*")
 		(sheetname "Root")
-		(sheetfile "auxiliary-pi-hat.kicad_sch")
+		(sheetfile "auxiliary-board.kicad_sch")
 		(attr through_hole)
 		(fp_line
@@
 		(property ki_fp_filters "R_*")
 		(sheetname "Root")
-		(sheetfile "auxiliary-pi-hat.kicad_sch")
+		(sheetfile "auxiliary-board.kicad_sch")
 		(attr smd)
 		(fp_line
@@
 		(property ki_fp_filters "R_*")
 		(sheetname "Root")
-		(sheetfile "auxiliary-pi-hat.kicad_sch")
+		(sheetfile "auxiliary-board.kicad_sch")
 		(attr smd)
 		(fp_line
@@
 		(property ki_fp_filters "Connector*:*_1x??_*")
 		(sheetname "Root")
-		(sheetfile "auxiliary-pi-hat.kicad_sch")
+		(sheetfile "auxiliary-board.kicad_sch")
 		(attr through_hole)
 		(fp_line
@@
 		(property ki_fp_filters "SOT?23*")
 		(sheetname "Root")
-		(sheetfile "auxiliary-pi-hat.kicad_sch")
+		(sheetfile "auxiliary-board.kicad_sch")
 		(attr smd)
 		(fp_line
@@
 		(property ki_fp_filters "Jumper* TestPoint*3Pads* TestPoint*Bridge*")
 		(sheetname "Root")
-		(sheetfile "auxiliary-pi-hat.kicad_sch")
+		(sheetfile "auxiliary-board.kicad_sch")
 		(zone_connect 1)
 		(attr exclude_from_pos_files exclude_from_bom)
@@
 		)
 		(sheetname "Root")
-		(sheetfile "auxiliary-pi-hat.kicad_sch")
+		(sheetfile "auxiliary-board.kicad_sch")
 		(attr through_hole)
 		(fp_rect
@@
 			(layers "*.Cu" "*.Mask")
 			(remove_unused_layers no)
-			(net 17 "SDA")
-			(pinfunction "SDA")
-			(pintype "bidirectional")
+			(net 18 "SCL")
+			(pinfunction "SCL")
+			(pintype "input")
 		)
 		(pad "5" thru_hole circle
@@
 			(layers "*.Cu" "*.Mask")
 			(remove_unused_layers no)
-			(net 18 "SCL")
-			(pinfunction "SCL")
-			(pintype "input")
+			(net 17 "SDA")
+			(pinfunction "SDA")
+			(pintype "bidirectional")
 		)
 		(pad "6" thru_hole circle
@@
 		)
 	)
-	(gr_text "ElectroPup\nAuxiliary Pi Hat\nmetaphasiclabs.com\nv1.0 : 10/2024"
+	(gr_text "ElectroPup\nAuxiliary Pi Hat\nmetaphasiclabs.com\nv1.1 : 10/2024"
 		(at 133.5 80.25 0)
 		(layer "B.SilkS")
@@
 	)
 	(segment
+		(start 155.74 75.92)
+		(end 158.28 78.46)
+		(width 0.35)
+		(layer "F.Cu")
+		(net 17)
+	)
+	(segment
 		(start 103.75 55.19575)
 		(end 101.91 53.35575)
@@
 	)
 	(segment
-		(start 158.28 75.92)
-		(end 154.92 75.92)
-		(width 0.25)
+		(start 154.92 75.92)
+		(end 155.74 75.92)
+		(width 0.35)
+		(layer "F.Cu")
+		(net 17)
+	)
+	(segment
+		(start 157.82 78)
+		(end 158.28 78.46)
+		(width 0.2)
 		(layer "F.Cu")
 		(net 17)
@@
 	)
 	(segment
+		(start 155.96 78.46)
+		(end 157.097 79.597)
+		(width 0.35)
+		(layer "F.Cu")
+		(net 18)
+	)
+	(segment
 		(start 104.45 54.95)
 		(end 104.45 53.35575)
@@
 	)
 	(segment
-		(start 158.28 78.46)
-		(end 155.96 78.46)
-		(width 0.25)
+		(start 158.903 79.597)
+		(end 159.5 79)
+		(width 0.35)
 		(layer "F.Cu")
 		(net 18)
@@
 	)
 	(segment
+		(start 157.097 79.597)
+		(end 158.903 79.597)
+		(width 0.35)
+		(layer "F.Cu")
+		(net 18)
+	)
+	(segment
 		(start 155.96 78.46)
 		(end 151.5 74)
@@
 		(layer "F.Cu")
 		(net 18)
+	)
+	(segment
+		(start 159.5 77.14)
+		(end 158.28 75.92)
+		(width 0.35)
+		(layer "F.Cu")
+		(net 18)
+	)
+	(segment
+		(start 159.5 79)
+		(end 159.5 77.14)
+		(width 0.35)
+		(layer "F.Cu")
+		(net 18)
