File: pcbs/auxiliary-board/auxiliary-board.kicad_sch (KiCad schematic)
At the start: 32 parts, among them J1 Conn_01x02, J10 Conn_01x03, J11 Conn_01x03, J2 Raspberry Pi - Hat Template -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, J3 Conn_01x03, J4 Conn_01x03, J5 Conn_01x03, J7 Conn_01x04, J8 Conn_02x04_Odd_Even, J9 Conn_01x05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

Commit message: cleanup
Connections:
- net SCL: now also MOD1.4 (SCL); no longer MOD1.5 (SCL)
- net SDA: now also MOD1.5 (SDA); no longer MOD1.4 (SDA)
Changed lines of the file:
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@@
-	)
-	(symbol
-		(lib_id "General:BNO055_Module")
-		(at 165.1 218.44 0)
-		(unit 1)
-		(exclude_from_sim no)
-		(in_bom yes)
-		(on_board yes)
-		(dnp no)
-		(fields_autoplaced yes)
-		(property "Reference" "MOD1"
-			(at 168.5641 201.93 0)
-			(effects
-				(font
-					(size 1.27 1.27)
-				)
-				(justify left)
-			)
-		)
-		(property "Value" "BNO055_Module"
-			(at 168.5641 204.47 0)
-			(effects
-				(font
-					(size 1.27 1.27)
-				)
-				(justify left)
-			)
-		)
-		(property "Footprint" "general:BNO055 Module"
-			(at 180.34 224.79 0)
-			(effects
-				(font
-					(size 1.27 1.27)
-				)
-				(hide yes)
-			)
-		)
-		(property "Datasheet" ""
-			(at 165.1 218.44 0)
-			(effects
-				(font
-					(size 1.27 1.27)
-				)
-				(hide yes)
-			)
-		)
-		(property "Description" ""
-			(at 165.1 218.44 0)
-			(effects
-				(font
-					(size 1.27 1.27)
-				)
-				(hide yes)
-			)
-		)
-		(pin "4"
-		)
-		(pin "7"
-		)
-		(pin "10"
-		)
-		(pin "9"
-		)
-		(pin "5"
-		)
-		(pin "1"
-		)
-		(pin "2"
-		)
-		(pin "3"
-		)
-		(pin "6"
-		)
-		(pin "8"
-		)
-		(instances
-			(project ""
-				(path "/312efdca-dfe3-4c27-a2ae-6c196f0be09d"
-					(reference "MOD1")
-					(unit 1)
-				)
-			)
-		)
 	)
 	(symbol
@@
 					(unit 1)
 				)
+			)
+		)
+	)
+	(symbol
+		(lib_id "General:BNO055_Module")
+		(at 165.1 218.44 0)
+		(unit 1)
+		(exclude_from_sim no)
+		(in_bom yes)
+		(on_board yes)
+		(dnp no)
+		(fields_autoplaced yes)
+		(property "Reference" "MOD1"
+			(at 168.5641 201.93 0)
+			(effects
+				(font
+					(size 1.27 1.27)
+				)
+				(justify left)
+			)
+		)
+		(property "Value" "BNO055_Module"
+			(at 168.5641 204.47 0)
+			(effects
+				(font
+					(size 1.27 1.27)
+				)
+				(justify left)
+			)
+		)
+		(property "Footprint" "general:BNO055 Module"
+			(at 180.34 224.79 0)
+			(effects
+				(font
+					(size 1.27 1.27)
+				)
+				(hide yes)
+			)
+		)
+		(property "Datasheet" ""
+			(at 165.1 218.44 0)
+			(effects
+				(font
+					(size 1.27 1.27)
+				)
+				(hide yes)
+			)
+		)
+		(property "Description" ""
+			(at 165.1 218.44 0)
+			(effects
+				(font
+					(size 1.27 1.27)
+				)
+				(hide yes)
+			)
+		)
+		(pin "4"
+		)
+		(pin "7"
+		)
+		(pin "10"
+		)
+		(pin "9"
+		)
+		(pin "5"
+		)
+		(pin "1"
+		)
+		(pin "2"
+		)
+		(pin "3"
+		)
+		(pin "6"
+		)
+		(pin "8"
+		)
+		(instances
+			(project "auxiliary-board"
+				(path "/312efdca-dfe3-4c27-a2ae-6c196f0be09d"
+					(reference "MOD1")
+					(unit 1)
+				)
